Commit message: commented stuff so that it does not work

File: roscon_gazebo/urdf/turret.xacro (robot description, xacro)
@@ -21,10 +21,10 @@
       </material>
 <xacro:macro name="inertia" params="mass">
-     <inertial>
+<!--     <inertial>
       <mass value="${mass}"/>
       <inertia  izz="${mass}" ixy="0.0"  ixz="0.0"
                 iyy="${mass}" iyz="0.0"
                 ixx="${mass}" />
-    </inertial>
+    </inertial>-->
 </xacro:macro>
 <link name="world"/>
@@ -43,5 +43,11 @@
     <material name="matbase"/>
     </visual>
-    <xacro:inertia mass="10"/>
+    <collision>
+      <origin xyz="0 0 0.25" rpy="0 0 0" />
+      <geometry>
+        <cylinder length="0.5" radius="0.025"/>
+      </geometry>
+    </collision>
+    <xacro:inertia mass="0.5"/>
   </link>
 <link name="turret/link1">
@@ -149,5 +155,5 @@
         </xacro:if>
     </xacro:macro>
-    <gazebo>
+<gazebo>
       <!-- Velocity or position control -->
       <xacro:control joint="joint1"/>
@@ -156,4 +162,13 @@
       <!-- Publish joint states anyway -->
       <plugin filename="ignition-gazebo-joint-state-publisher-system" name="ignition::gazebo::systems::JointStatePublisher"/>
+      <!-- Publish pose of this model -->
+      <plugin
+            filename="ignition-gazebo-pose-publisher-system"
+            name="ignition::gazebo::systems::PosePublisher">
+            <publish_link_pose>false</publish_link_pose>
+            <publish_collision_pose>false</publish_collision_pose>
+            <publish_visual_pose>false</publish_visual_pose>
+            <publish_nested_model_pose>true</publish_nested_model_pose>
+        </plugin>
     </gazebo>
  <gazebo reference="turret/tool0">

Commit message: more comments

File: roscon_gazebo/urdf/turret.xacro (robot description, xacro)
@@ -43,10 +43,10 @@
     <material name="matbase"/>
     </visual>
-    <collision>
+<!--    <collision>
       <origin xyz="0 0 0.25" rpy="0 0 0" />
       <geometry>
         <cylinder length="0.5" radius="0.025"/>
       </geometry>
-    </collision>
+    </collision>-->
     <xacro:inertia mass="0.5"/>
   </link>

Commit message: typos / launch XML example

File: roscon_gazebo/urdf/turret.xacro (robot description, xacro)
@@ -28,4 +28,5 @@
     </inertial>-->
 </xacro:macro>
+<!--
 <link name="world"/>
 <joint name="base_link" type="fixed">
@@ -33,5 +34,5 @@
     <child link="turret/base_link" />
     <origin xyz="$(arg x) $(arg y) 0.0" />
-</joint>
+</joint>-->
 <!-- Links -->
   <link name="turret/base_link">

Commit message: explicit GazeboBridge

File: roscon_gazebo/urdf/turret.xacro (robot description, xacro)
@@ -28,6 +28,5 @@
     </inertial>-->
 </xacro:macro>
-<!--
-<link name="world"/>
+<!--<link name="world"/>
 <joint name="base_link" type="fixed">
     <parent link="world" />
